File: hardware/cm4-hsio.kicad_sch (KiCad schematic)
At the start: 3 parts, among them J1 DF40C-100DP-0.4V_51_

Commit message: minor schematic revisions
Connections:
- net USB3_0_C_N: no longer names the net of J1.40
- net USB3_0_C_P: no longer names the net of J1.42
- net USB3_0_D0_N: no longer names the net of J1.28
- net USB3_0_D0_P: no longer names the net of J1.30
- net USB3_0_D1_N: no longer names the net of J1.34
- net USB3_0_D1_P: no longer names the net of J1.36
- no-connect marks 20 -> 24
Other:
- note added: "USB3_0_C_N"
- note added: "USB3_0_C_P"
- note added: "USB3_0_D0_N"
- note added: "USB3_0_D0_P"
- note added: "USB3_0_D1_N"
- note added: "USB3_0_D1_P"
Changed lines of the file:
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@@
+		)
+	)
+	(text "USB3_0_D0_P"
+		(exclude_from_sim no)
+		(at 91.44 63.5 0)
+		(effects
+			(font
+				(size 1.27 1.27)
+			)
+			(justify left bottom)
 		)
 	)
@@
 		)
 	)
+	(text "USB3_0_D0_N"
+		(exclude_from_sim no)
+		(at 91.44 60.96 0)
+		(effects
+			(font
+				(size 1.27 1.27)
+			)
+			(justify left bottom)
+		)
+	)
+	(text "USB3_0_D1_P"
+		(exclude_from_sim no)
+		(at 91.44 71.12 0)
+		(effects
+			(font
+				(size 1.27 1.27)
+			)
+			(justify left bottom)
+		)
+	)
 	(text "DDMI1"
 		(exclude_from_sim no)
@@
 				(bold yes)
 			)
+		)
+	)
+	(text "USB3_0_D1_N"
+		(exclude_from_sim no)
+		(at 91.44 68.58 0)
+		(effects
+			(font
+				(size 1.27 1.27)
+			)
+			(justify left bottom)
 		)
 	)
@@
 		)
 	)
+	(text "USB3_0_C_P"
+		(exclude_from_sim no)
+		(at 91.44 78.74 0)
+		(effects
+			(font
+				(size 1.27 1.27)
+			)
+			(justify left bottom)
+		)
+	)
 	(text "Diff tuned to 17mm\nDiff Skew tuned\n"
 		(exclude_from_sim no)
@@
 		)
 	)
+	(text "USB3_0_C_N"
+		(exclude_from_sim no)
+		(at 91.44 76.2 0)
+		(effects
+			(font
+				(size 1.27 1.27)
+			)
+			(justify left bottom)
+		)
+	)
 	(text "Diff tuned to 28mm\nDiff Skew tuned\n"
 		(exclude_from_sim no)
@@
 	)
 	(no_connect
-		(at 102.87 68.58)
-	)
-	(no_connect
-		(at 102.87 76.2)
-	)
-	(no_connect
 		(at 62.23 101.6)
 	)
@@
 	)
 	(no_connect
-		(at 102.87 78.74)
+		(at 87.63 78.74)
+	)
+	(no_connect
+		(at 87.63 63.5)
 	)
 	(no_connect
@@
 	)
 	(no_connect
-		(at 102.87 71.12)
+		(at 87.63 76.2)
 	)
 	(no_connect
-		(at 102.87 60.96)
+		(at 62.23 147.32)
+	)
+	(no_connect
+		(at 87.63 68.58)
 	)
 	(no_connect
@@
 	)
 	(no_connect
+		(at 87.63 71.12)
+	)
+	(no_connect
 		(at 62.23 81.28)
 	)
@@
 	)
 	(no_connect
+		(at 87.63 144.78)
+	)
+	(no_connect
 		(at 62.23 88.9)
+	)
+	(no_connect
+		(at 62.23 144.78)
+	)
+	(no_connect
+		(at 87.63 147.32)
 	)
 	(no_connect
@@
 	)
 	(no_connect
+		(at 87.63 60.96)
+	)
+	(no_connect
 		(at 62.23 93.98)
 	)
@@
 		(at 62.23 91.44)
 	)
-	(no_connect
-		(at 102.87 63.5)
-	)
 	(bus_entry
 		(at 102.87 93.98)
@@
 	)
 	(bus_entry
-		(at 102.87 55.88)
-		(size 2.54 2.54)
-		(stroke
-			(width 0)
-			(type default)
-		)
-	)
-	(bus_entry
 		(at 102.87 116.84)
 		(size 2.54 2.54)
@@
 		)
 	)
-	(wire
-		(pts
-			(xy 87.63 71.12) (xy 102.87 71.12)
-		)
-		(stroke
-			(width 0)
-			(type default)
-		)
-	)
 	(bus
 		(pts
@@
 		)
 	)
-	(wire
-		(pts
-			(xy 87.63 78.74) (xy 102.87 78.74)
-		)
-		(stroke
-			(width 0)
-			(type default)
-		)
-	)
 	(bus
 		(pts
@@
 	(wire
 		(pts
-			(xy 87.63 60.96) (xy 102.87 60.96)
-		)
-		(stroke
-			(width 0)
-			(type default)
-		)
-	)
-	(wire
-		(pts
 			(xy 46.99 33.02) (xy 62.23 33.02)
 		)
@@
 	(wire
 		(pts
-			(xy 87.63 76.2) (xy 102.87 76.2)
-		)
-		(stroke
-			(width 0)
-			(type default)
-		)
-	)
-	(wire
-		(pts
 			(xy 87.63 121.92) (xy 102.87 121.92)
 		)
@@
 	(wire
 		(pts
-			(xy 87.63 63.5) (xy 102.87 63.5)
-		)
-		(stroke
-			(width 0)
-			(type default)
-		)
-	)
-	(wire
-		(pts
 			(xy 59.69 66.04) (xy 59.69 73.66)
 		)
@@
 	(wire
 		(pts
-			(xy 87.63 68.58) (xy 102.87 68.58)
-		)
-		(stroke
-			(width 0)
-			(type default)
-		)
-	)
-	(wire
-		(pts
 			(xy 87.63 81.28) (xy 90.17 81.28)
 		)
@@
 			(width 0)
 			(type default)
-		)
-	)
-	(label "USB3_0_D0_P"
-		(at 102.87 63.5 180)
-		(effects
-			(font
-				(size 1.27 1.27)
-			)
-			(justify right bottom)
 		)
 	)
@@
 		)
 	)
-	(label "USB3_0_D1_P"
-		(at 102.87 71.12 180)
-		(effects
-			(font
-				(size 1.27 1.27)
-			)
-			(justify right bottom)
-		)
-	)
-	(label "USB3_0_C_N"
-		(at 102.87 76.2 180)
-		(effects
-			(font
-				(size 1.27 1.27)
-			)
-			(justify right bottom)
-		)
-	)
 	(label "LVDS1_D1_N"
 		(at 57.15 129.54 180)
@@
 		)
 	)
-	(label "USB3_0_D1_N"
-		(at 102.87 68.58 180)
-		(effects
-			(font
-				(size 1.27 1.27)
-			)
-			(justify right bottom)
-		)
-	)
 	(label "DDMI0_TX2_N"
 		(at 102.87 116.84 180)
@@
 		)
 	)
-	(label "USB3_0_C_P"
-		(at 102.87 78.74 180)
-		(effects
-			(font
-				(size 1.27 1.27)
-			)
-			(justify right bottom)
-		)
-	)
 	(label "DDMI0_SCL"
 		(at 102.87 152.4 180)
@@
 		(effects
 			(font
-				(size 1.27 1.27)
-			)
-			(justify right bottom)
-		)
-	)
-	(label "USB3_0_D0_N"
-		(at 102.87 60.96 180)
-		(effects
-			(font
