File: hardware/gpio.kicad_sch (KiCad schematic)
At the start: 11 parts, among them U4 GateMate-CCGM1A1

Commit message: minor schematic revisions
Parts:
- removed R115: dnp, Resistor_SMD:R_0402_1005Metric, symbol Device:R_Small
- removed R116: 0R, Resistor_SMD:R_0402_1005Metric, symbol Device:R_Small
Connections:
- net SDRAM_A1 is gone; now on net SD_DAT2: U4.A3 (IO_NA_A0)
- net SDRAM_A10 is gone; now on net SD_DAT1: U4.B4 (IO_NA_B1)
- net SDRAM_VCC is gone; now on net GPIO_VREF: C86.1, C87.1, C88.1, C89.1, C90.1, C91.1, C92.1, C93.1, U4.A5 (VDD_NA), U4.B10 (VDD_NB), U4.B13 (VDD_NB), U4.B7 (VDD_NA), U4.E10 (VDD_NB), U4.E12 (VDD_NB), U4.E6 (VDD_NA), U4.E8 (VDD_NA), U4.F11 (VDD_NB), U4.F7 (VDD_NA)
- net GPIO11: now also U4.D10 (IO_NB_A1); no longer U4.C11 (IO_NB_B3)
- net GPIO13: now also U4.C14 (IO_NB_B8); no longer U4.D13 (IO_NB_A6)
- net GPIO14: now also U4.B6 (IO_NA_B4); no longer U4.A6 (IO_NA_A4)
- net GPIO15: now also U4.A6 (IO_NA_A4); no longer U4.B6 (IO_NA_B4)
- net GPIO17: now also U4.D8 (IO_NA_B6); no longer U4.C8 (IO_NA_A6)
- net GPIO18: now also U4.B8 (IO_NA_B7); no longer U4.A8 (IO_NA_A7)
- net GPIO19: now also U4.D13 (IO_NB_A6); no longer U4.C14 (IO_NB_B8)
- net GPIO23: now also U4.A8 (IO_NA_A7); no longer U4.B8 (IO_NA_B7)
- net GPIO24: now also U4.B9 (IO_NB_A0); no longer U4.A9 (IO_NB_B0)
- net GPIO25: now also U4.A9 (IO_NB_B0); no longer U4.B9 (IO_NB_A0)
- net GPIO4: now also U4.C8 (IO_NA_A6); no longer U4.D8 (IO_NA_B6)
- net GPIO9: now also U4.C11 (IO_NB_B3); no longer U4.D10 (IO_NB_A1)
- net SD_DAT1: no longer U4.D12 (IO_NB_A5)
- net SD_DAT2: no longer U4.C5 (IO_NA_B2)
- net FAN_PWM: no longer names the net of U4.D11 (IO_NB_A3)
- net SDRAM_A2 renamed SDA0
- new net SCL0: U4.C5 (IO_NA_B2)
- no-connect marks 0 -> 2
