File: hardware/ulx5m-gs.kicad_sch (KiCad schematic)
At the start: 4 parts

Commit message: minor schematic revisions
Other:
- sheet gpdi-ram renamed memory
- sheet cm4-gpio ports: added none; removed FAN_PWM, GPIO_VREF, ID_SC, ID_SD
- sheet ethernet ports: added none; removed ID_SC, ID_SD, {DDMI1}, {I2C}, {SD}
- sheet gpio ports: added {I2C}; removed FAN_PWM, GPIO_VREF
- sheet lvds ports: added {DDMI1}; removed none
- sheet memory: file ram.kicad_sch -> memory.kicad_sch
- note removed: "4HIGH bit SD"
